File: 0.1/compact/ferris.kicad_pcb (KiCad board)
At the start: 2 copper layers, 208.7 x 86.7 mm, 102 parts, among them J1 USB C, K0_0 KEYSW, K0_1 KEYSW, K0_2 KEYSW, K0_3 KEYSW, K0_4 KEYSW, K0_5 KEYSW, K0_6 KEYSW, K0_7 KEYSW, K0_8 KEYSW, K0_9 KEYSW, K1_0 KEYSW, K1_1 KEYSW, K1_2 KEYSW, K1_3 KEYSW, K1_4 KEYSW, K1_5 KEYSW, K1_6 KEYSW, K1_7 KEYSW, K1_8 KEYSW, K1_9 KEYSW, K2_0 KEYSW, K2_1 KEYSW, K2_2 KEYSW, K2_3 KEYSW, K2_4 KEYSW, K2_5 KEYSW, K2_6 KEYSW, K2_7 KEYSW, K2_8 KEYSW, K2_9 KEYSW, K3_3 KEYSW, K3_4 KEYSW, K3_5 KEYSW, K3_6 KEYSW, SW1 SW_PUSH, U1 ATmega32U4-AU, U2 MCP23017_SO, Y1 Crystal

Commit message: Temporarily increase solder mask clearance in order to move traces.
The solder mask clearance should be set back to 0.05mm after the traces have
been moved.
Other:
- rule pad_to_mask_clearance: 0.05 -> 0.61
Changed lines of the file:
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@@
     (36 B.SilkS user hide)
     (37 F.SilkS user hide)
-    (38 B.Mask user hide)
-    (39 F.Mask user hide)
+    (38 B.Mask user)
+    (39 F.Mask user)
     (40 Dwgs.User user hide)
     (41 Cmts.User user hide)
@@
     (pad_size 1.524 1.524)
     (pad_drill 0.762)
-    (pad_to_mask_clearance 0.05)
+    (pad_to_mask_clearance 0.61)
     (aux_axis_origin 0 0)
     (visible_elements FFFFFFFF)

Commit message: Revert "Temporarily increase solder mask clearance in order to move traces."
This reverts commit 0fd1c5d82cd2eb1b42baabec2bdd6d8ffa0e2c2a.
Other:
- rule pad_to_mask_clearance: 0.61 -> 0.05
Changed lines of the file:
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@@
     (36 B.SilkS user hide)
     (37 F.SilkS user hide)
-    (38 B.Mask user)
-    (39 F.Mask user)
+    (38 B.Mask user hide)
+    (39 F.Mask user hide)
     (40 Dwgs.User user hide)
     (41 Cmts.User user hide)
@@
     (pad_size 1.524 1.524)
     (pad_drill 0.762)
-    (pad_to_mask_clearance 0.61)
+    (pad_to_mask_clearance 0.05)
     (aux_axis_origin 0 0)
     (visible_elements FFFFFFFF)
